File: bee/bee.kicad_pcb (KiCad board)
At the start: 2 copper layers, 29 x 53.3 mm, 12 parts, among them J1 Conn_01x02_Male, J2 Conn_01x02_Male, J3 Conn_01x02_Male, J4 Conn_01x02_Male

Commit message: Add sch symbols for labels, update PCB accordingly.
Parts:
- removed REF** (x2): Text_U_B+_Silkscreen, Symbol-emt:Text_U_B+_Silkscreen
- removed REF** (x2): Text_U_B-_Silkscreen, Symbol-emt:Text_U_B-_Silkscreen
- removed REF** (x2): Text_U_B2_Silkscreen, Symbol-emt:Text_U_B2_Silkscreen
- removed REF** (x2): Symbol_GND_Silkscreen, Symbol-emt:Symbol_GND_Silkscreen
- added H1: Silkscreen_Label, Symbol-emt:Text_U_B+_Silkscreen, F.Cu at (75.2, 91.4)
- added H2: Silkscreen_Label, Symbol-emt:Text_U_B+_Silkscreen, F.Cu at (101.1, 91.4)
- added H3: Silkscreen_Label, Symbol-emt:Text_U_B-_Silkscreen, F.Cu at (75.2, 94.0)
- added H4: Silkscreen_Label, Symbol-emt:Text_U_B-_Silkscreen, F.Cu at (101.1, 94.0)
- added H5: Silkscreen_Label, Symbol-emt:Text_U_B2_Silkscreen, F.Cu at (75.2, 137.2)
- added H6: Silkscreen_Label, Symbol-emt:Text_U_B2_Silkscreen, F.Cu at (101.1, 137.2)
- added H7: Silkscreen_Label, Symbol-emt:Symbol_GND_Silkscreen, F.Cu at (75.7, 139.7)
- added H8: Silkscreen_Label, Symbol-emt:Symbol_GND_Silkscreen, F.Cu at (102.1, 139.7)
Changed lines of the file:
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@@
-(kicad_pcb (version 20171130) (host pcbnew 5.0.2+dfsg1-1~bpo9+1)
+(kicad_pcb (version 20171130) (host pcbnew "(5.1.0)-1")
   (general
     (thickness 1.6)
@@
     (zone_45_only no)
     (trace_min 0.2)
-    (segment_width 0.2)
-    (edge_width 0.15)
     (via_size 0.8)
     (via_drill 0.4)
@@
     (uvia_min_size 0.2)
     (uvia_min_drill 0.1)
+    (edge_width 0.15)
+    (segment_width 0.2)
     (pcb_text_width 0.3)
     (pcb_text_size 1.5 1.5)
@@
     (solder_mask_min_width 0.25)
     (aux_axis_origin 0 0)
-    (visible_elements FFFFFF7F)
+    (visible_elements 7FFFFFFF)
     (pcbplotparams
       (layerselection 0x010fc_ffffffff)
@@
     (tags "Voltage Label Betriebsspannung")
     (attr virtual)
-    (fp_text reference REF** (at 0 1.65) (layer F.SilkS) hide
-      (effects (font (size 1 1) (thickness 0.15)))
-    )
-    (fp_text value Text_U_B+_Silkscreen (at 0 -1.5) (layer F.Fab) hide
+    (fp_text reference H1 (at 0 1.65) (layer F.SilkS) hide
+      (effects (font (size 1 1) (thickness 0.15)))
+    )
+    (fp_text value Silkscreen_Label (at 0 -1.5) (layer F.Fab) hide
       (effects (font (size 1 1) (thickness 0.15)))
     )
@@
     (fp_text user U (at 0 0) (layer F.SilkS)
       (effects (font (size 1 1) (thickness 0.15)))
+    )
+  )
+  (module Symbol-emt:Text_U_B+_Silkscreen (layer F.Cu)
+    (at 101.092 91.44)
+    (descr "Voltage Label Betriebsspannung")
+    (tags "Voltage Label Betriebsspannung")
+    (attr virtual)
+    (fp_text reference H2 (at 0 1.65) (layer F.SilkS) hide
+      (effects (font (size 1 1) (thickness 0.15)))
+    )
+    (fp_text value Silkscreen_Label (at 0 -1.5) (layer F.Fab) hide
+      (effects (font (size 1 1) (thickness 0.15)))
+    )
+    (fp_text user U (at 0 0) (layer F.SilkS)
+      (effects (font (size 1 1) (thickness 0.15)))
+    )
+    (fp_text user B+ (at 1.2 0.5) (layer F.SilkS)
+      (effects (font (size 0.7 0.7) (thickness 0.1)))
     )
   )
@@
     (tags "Voltage Label Betriebsspannung")
     (attr virtual)
-    (fp_text reference REF** (at 0 1.65) (layer F.SilkS) hide
-      (effects (font (size 1 1) (thickness 0.15)))
-    )
-    (fp_text value Text_U_B-_Silkscreen (at 0 -1.5) (layer F.Fab) hide
+    (fp_text reference H3 (at 0 1.65) (layer F.SilkS) hide
+      (effects (font (size 1 1) (thickness 0.15)))
+    )
+    (fp_text value Silkscreen_Label (at 0 -1.5) (layer F.Fab) hide
       (effects (font (size 1 1) (thickness 0.15)))
     )
@@
     (fp_text user U (at 0 0) (layer F.SilkS)
       (effects (font (size 1 1) (thickness 0.15)))
+    )
+  )
+  (module Symbol-emt:Text_U_B-_Silkscreen (layer F.Cu)
+    (at 101.092 93.98)
+    (descr "Voltage Label Betriebsspannung")
+    (tags "Voltage Label Betriebsspannung")
+    (attr virtual)
+    (fp_text reference H4 (at 0 1.65) (layer F.SilkS) hide
+      (effects (font (size 1 1) (thickness 0.15)))
+    )
+    (fp_text value Silkscreen_Label (at 0 -1.5) (layer F.Fab) hide
+      (effects (font (size 1 1) (thickness 0.15)))
+    )
+    (fp_text user U (at 0 0) (layer F.SilkS)
+      (effects (font (size 1 1) (thickness 0.15)))
+    )
+    (fp_text user B- (at 1.2 0.5) (layer F.SilkS)
+      (effects (font (size 0.7 0.7) (thickness 0.1)))
     )
   )
@@
     (tags "Voltage Label Betriebsspannung")
     (attr virtual)
-    (fp_text reference REF** (at 0 1.65) (layer F.SilkS) hide
-      (effects (font (size 1 1) (thickness 0.15)))
-    )
-    (fp_text value Text_U_B2_Silkscreen (at 0 -1.5) (layer F.Fab) hide
+    (fp_text reference H5 (at 0 1.65) (layer F.SilkS) hide
+      (effects (font (size 1 1) (thickness 0.15)))
+    )
+    (fp_text value Silkscreen_Label (at 0 -1.5) (layer F.Fab) hide
+      (effects (font (size 1 1) (thickness 0.15)))
+    )
+    (fp_text user U (at 0 0) (layer F.SilkS)
+      (effects (font (size 1 1) (thickness 0.15)))
+    )
+    (fp_text user B2 (at 1.1 0.5) (layer F.SilkS)
+      (effects (font (size 0.7 0.7) (thickness 0.1)))
+    )
+  )
+  (module Symbol-emt:Text_U_B2_Silkscreen (layer F.Cu)
+    (at 101.092 137.16)
+    (descr "Voltage Label Betriebsspannung")
+    (tags "Voltage Label Betriebsspannung")
+    (attr virtual)
+    (fp_text reference H6 (at 0 1.65) (layer F.SilkS) hide
+      (effects (font (size 1 1) (thickness 0.15)))
+    )
+    (fp_text value Silkscreen_Label (at 0 -1.5) (layer F.Fab) hide
       (effects (font (size 1 1) (thickness 0.15)))
     )
@@
     (tags "Symbol GND")
     (attr virtual)
-    (fp_text reference REF** (at 0 1.6) (layer F.SilkS) hide
-      (effects (font (size 1 1) (thickness 0.15)))
-    )
-    (fp_text value Symbol_GND_Silkscreen (at 0 -0.75) (layer F.Fab) hide
-      (effects (font (size 1 1) (thickness 0.15)))
-    )
+    (fp_text reference H7 (at 0 1.6) (layer F.SilkS) hide
+      (effects (font (size 1 1) (thickness 0.15)))
+    )
+    (fp_text value Silkscreen_Label (at 0 -0.75) (layer F.Fab) hide
+      (effects (font (size 1 1) (thickness 0.15)))
+    )
+    (fp_line (start -0.5 0.8) (end 0.5 0.8) (layer F.SilkS) (width 0.25))
     (fp_line (start 0 0.8) (end 0 0) (layer F.SilkS) (width 0.15))
-    (fp_line (start -0.5 0.8) (end 0.5 0.8) (layer F.SilkS) (width 0.25))
-  )
-  (module Symbol-emt:Text_U_B+_Silkscreen (layer F.Cu)
-    (at 101.092 91.44)
-    (descr "Voltage Label Betriebsspannung")
-    (tags "Voltage Label Betriebsspannung")
-    (attr virtual)
-    (fp_text reference REF** (at 0 1.65) (layer F.SilkS) hide
-      (effects (font (size 1 1) (thickness 0.15)))
-    )
-    (fp_text value Text_U_B+_Silkscreen (at 0 -1.5) (layer F.Fab) hide
-      (effects (font (size 1 1) (thickness 0.15)))
-    )
-    (fp_text user B+ (at 1.2 0.5) (layer F.SilkS)
-      (effects (font (size 0.7 0.7) (thickness 0.1)))
-    )
-    (fp_text user U (at 0 0) (layer F.SilkS)
-      (effects (font (size 1 1) (thickness 0.15)))
-    )
-  )
-  (module Symbol-emt:Text_U_B-_Silkscreen (layer F.Cu)
-    (at 101.092 93.98)
-    (descr "Voltage Label Betriebsspannung")
-    (tags "Voltage Label Betriebsspannung")
-    (attr virtual)
-    (fp_text reference REF** (at 0 1.65) (layer F.SilkS) hide
-      (effects (font (size 1 1) (thickness 0.15)))
-    )
-    (fp_text value Text_U_B-_Silkscreen (at 0 -1.5) (layer F.Fab) hide
-      (effects (font (size 1 1) (thickness 0.15)))
-    )
-    (fp_text user B- (at 1.2 0.5) (layer F.SilkS)
-      (effects (font (size 0.7 0.7) (thickness 0.1)))
-    )
-    (fp_text user U (at 0 0) (layer F.SilkS)
-      (effects (font (size 1 1) (thickness 0.15)))
-    )
-  )
-  (module Symbol-emt:Text_U_B2_Silkscreen (layer F.Cu)
-    (at 101.092 137.16)
-    (descr "Voltage Label Betriebsspannung")
-    (tags "Voltage Label Betriebsspannung")
-    (attr virtual)
-    (fp_text reference REF** (at 0 1.65) (layer F.SilkS) hide
-      (effects (font (size 1 1) (thickness 0.15)))
-    )
-    (fp_text value Text_U_B2_Silkscreen (at 0 -1.5) (layer F.Fab) hide
-      (effects (font (size 1 1) (thickness 0.15)))
-    )
-    (fp_text user B2 (at 1.1 0.5) (layer F.SilkS)
-      (effects (font (size 0.7 0.7) (thickness 0.1)))
-    )
-    (fp_text user U (at 0 0) (layer F.SilkS)
-      (effects (font (size 1 1) (thickness 0.15)))
-    )
   )
   (module Symbol-emt:Symbol_GND_Silkscreen (layer F.Cu)
@@
     (tags "Symbol GND")
     (attr virtual)
-    (fp_text reference REF** (at 0 1.6) (layer F.SilkS) hide
-      (effects (font (size 1 1) (thickness 0.15)))
-    )
-    (fp_text value Symbol_GND_Silkscreen (at 0 -0.75) (layer F.Fab) hide
-      (effects (font (size 1 1) (thickness 0.15)))
-    )
+    (fp_text reference H8 (at 0 1.6) (layer F.SilkS) hide
+      (effects (font (size 1 1) (thickness 0.15)))
+    )
+    (fp_text value Silkscreen_Label (at 0 -0.75) (layer F.Fab) hide
+      (effects (font (size 1 1) (thickness 0.15)))
+    )
