File: bee/bee.kicad_pcb (KiCad board)
At the start: 2 copper layers, 29 x 53.3 mm, 16 parts, among them J1 Conn_01x02_Male, J2 Conn_01x02_Male, J3 Conn_01x02_Male, J4 Conn_01x02_Male

Commit message: Relabel as bee specific.
Parts:
- H1, H2: footprint Symbol-emt:Text_U_B+_Silkscreen -> Symbol-bee:Text_U_B+_Silkscreen
- H3, H4: footprint Symbol-emt:Text_U_B-_Silkscreen -> Symbol-bee:Text_U_B-_Silkscreen
- H5, H6: footprint Symbol-emt:Text_U_B2_Silkscreen -> Symbol-bee:Text_U_B2_Silkscreen
- H7, H8: footprint Symbol-emt:Symbol_GND_Silkscreen -> Symbol-bee:Symbol_GND_Silkscreen
Changed lines of the file:
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@@
     )
   )
-  (module Symbol-emt:Text_U_B+_Silkscreen (layer F.Cu)
+  (module Symbol-bee:Text_U_B+_Silkscreen (layer F.Cu)
     (at 75.184 91.44)
     (descr "Voltage Label Betriebsspannung")
@@
     )
   )
-  (module Symbol-emt:Text_U_B+_Silkscreen (layer F.Cu)
+  (module Symbol-bee:Text_U_B+_Silkscreen (layer F.Cu)
     (at 101.092 91.44)
     (descr "Voltage Label Betriebsspannung")
@@
     )
   )
-  (module Symbol-emt:Text_U_B-_Silkscreen (layer F.Cu)
+  (module Symbol-bee:Text_U_B-_Silkscreen (layer F.Cu)
     (at 75.184 93.98)
     (descr "Voltage Label Betriebsspannung")
@@
     )
   )
-  (module Symbol-emt:Text_U_B-_Silkscreen (layer F.Cu)
+  (module Symbol-bee:Text_U_B-_Silkscreen (layer F.Cu)
     (at 101.092 93.98)
     (descr "Voltage Label Betriebsspannung")
@@
     )
   )
-  (module Symbol-emt:Text_U_B2_Silkscreen (layer F.Cu)
+  (module Symbol-bee:Text_U_B2_Silkscreen (layer F.Cu)
     (at 75.184 137.16)
     (descr "Voltage Label Betriebsspannung")
@@
     )
   )
-  (module Symbol-emt:Text_U_B2_Silkscreen (layer F.Cu)
+  (module Symbol-bee:Text_U_B2_Silkscreen (layer F.Cu)
     (at 101.092 137.16)
     (descr "Voltage Label Betriebsspannung")
@@
     )
   )
-  (module Symbol-emt:Symbol_GND_Silkscreen (layer F.Cu)
+  (module Symbol-bee:Symbol_GND_Silkscreen (layer F.Cu)
     (at 75.692 139.7)
     (descr "Symbol GND")
@@
     (fp_line (start 0 0.8) (end 0 0) (layer F.SilkS) (width 0.15))
   )
-  (module Symbol-emt:Symbol_GND_Silkscreen (layer F.Cu)
+  (module Symbol-bee:Symbol_GND_Silkscreen (layer F.Cu)
     (at 102.108 139.7)
     (descr "Symbol GND")
